File: KiCad/isa_backplane.kicad_sch (KiCad schematic)
At the start: 67 parts, among them P1 POWER, P2 POWER_SW, P3 POWER_LED, SW1 POWER, U1 74HCT74, U2 74HCT14, U3 LM7905CT

Commit message: Move resistor arrays to the bottom
Parts:
- removed RR5: 4.7k, my_components:Conn_SIL6, symbol isa_backplane-rescue:RR5
- added C28: 10uF, My_Components:Cap_Tant_508, symbol isa_backplane-rescue:CP1
- added RR5: 4.7k, My_Components:Conn_SIL5, symbol my_components:RR4
- renumbered BUS8 to BUS6, BUS9 to BUS7, BUS6 to BUS8, BUS7 to BUS9
Connections:
- net +5V: now also RR5.1 (COM)
- net -12V: now also C28.2
- net GND: now also C28.1
- net ~{IOR}: now also RR5.5
- net ~{IOW}: now also RR5.4
- net ~{MEMR}: now also RR5.3
- net ~{MEMW}: now also RR5.2
- no-connect marks 8 -> 7
Changed lines of the file:
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@@
   (junction (at -102.87 229.87) (diameter 0) (color 0 0 0 0)
   )
+  (junction (at -116.84 252.73) (diameter 0) (color 0 0 0 0)
+  )
   (junction (at -85.09 240.03) (diameter 0) (color 0 0 0 0)
   )
@@
   (junction (at 276.86 137.16) (diameter 0) (color 0 0 0 0)
   )
+  (junction (at -116.84 240.03) (diameter 0) (color 0 0 0 0)
+  )
   (junction (at 264.16 210.82) (diameter 0) (color 0 0 0 0)
   )
@@
   )
   (no_connect (at 405.13 106.68))
-  (no_connect (at 238.76 228.6))
   (no_connect (at 378.46 33.02))
   (no_connect (at 342.9 50.8))
@@
     (stroke (width 0) (type default))
   )
+  (wire (pts (xy -107.95 252.73) (xy -107.95 250.19))
+    (stroke (width 0) (type default))
+  )
   (wire (pts (xy 289.56 149.86) (xy 294.64 149.86))
     (stroke (width 0) (type default))
@@
     (stroke (width 0) (type default))
   )
+  (wire (pts (xy -116.84 240.03) (xy -107.95 240.03))
+    (stroke (width 0) (type default))
+  )
   (wire (pts (xy 106.68 121.92) (xy 96.52 121.92))
     (stroke (width 0) (type default))
@@
     (stroke (width 0) (type default))
   )
-  (wire (pts (xy 236.22 226.06) (xy 236.22 220.98))
+  (wire (pts (xy 238.76 226.06) (xy 238.76 220.98))
     (stroke (width 0) (type default))
   )
@@
     (stroke (width 0) (type default))
   )
+  (wire (pts (xy -107.95 240.03) (xy -107.95 242.57))
+    (stroke (width 0) (type default))
+  )
   (wire (pts (xy 106.68 175.26) (xy 96.52 175.26))
     (stroke (width 0) (type default))
@@
     (stroke (width 0) (type default))
   )
-  (wire (pts (xy 236.22 220.98) (xy 213.36 220.98))
+  (wire (pts (xy 238.76 220.98) (xy 213.36 220.98))
     (stroke (width 0) (type default))
   )
@@
     (stroke (width 0) (type default))
   )
-  (wire (pts (xy 238.76 236.22) (xy 231.14 236.22))
+  (wire (pts (xy 238.76 233.68) (xy 231.14 233.68))
     (stroke (width 0) (type default))
   )
@@
     (stroke (width 0) (type default))
   )
-  (wire (pts (xy 238.76 226.06) (xy 236.22 226.06))
-    (stroke (width 0) (type default))
-  )
   (wire (pts (xy -69.85 252.73) (xy -69.85 250.19))
     (stroke (width 0) (type default))
@@
     (stroke (width 0) (type default))
   )
-  (wire (pts (xy 238.76 238.76) (xy 231.14 238.76))
+  (wire (pts (xy 238.76 236.22) (xy 231.14 236.22))
     (stroke (width 0) (type default))
   )
@@
     (stroke (width 0) (type default))
   )
-  (wire (pts (xy 238.76 233.68) (xy 231.14 233.68))
+  (wire (pts (xy 238.76 231.14) (xy 231.14 231.14))
     (stroke (width 0) (type default))
   )
@@
     (stroke (width 0) (type default))
   )
+  (wire (pts (xy -116.84 252.73) (xy -107.95 252.73))
+    (stroke (width 0) (type default))
+  )
   (wire (pts (xy 170.18 195.58) (xy 180.34 195.58))
     (stroke (width 0) (type default))
@@
     (stroke (width 0) (type default))
   )
-  (wire (pts (xy 238.76 231.14) (xy 231.14 231.14))
+  (wire (pts (xy 238.76 228.6) (xy 231.14 228.6))
     (stroke (width 0) (type default))
   )
@@
     (effects (font (size 1.524 1.524)) (justify right bottom))
   )
-  (label "~{IOR}" (at 231.14 238.76 0) (fields_autoplaced)
+  (label "~{IOR}" (at 231.14 236.22 0) (fields_autoplaced)
     (effects (font (size 1.524 1.524)) (justify left bottom))
   )
@@
     (effects (font (size 1.524 1.524)) (justify left bottom))
   )
-  (label "~{IOW}" (at 231.14 236.22 0) (fields_autoplaced)
+  (label "~{IOW}" (at 231.14 233.68 0) (fields_autoplaced)
     (effects (font (size 1.524 1.524)) (justify left bottom))
   )
@@
     (effects (font (size 1.524 1.524)) (justify right bottom))
   )
-  (label "~{MEMW}" (at 231.14 231.14 0) (fields_autoplaced)
+  (label "~{MEMW}" (at 231.14 228.6 0) (fields_autoplaced)
     (effects (font (size 1.524 1.524)) (justify left bottom))
   )
@@
     (effects (font (size 1.524 1.524)) (justify right bottom))
   )
-  (label "~{MEMR}" (at 231.14 233.68 0) (fields_autoplaced)
+  (label "~{MEMR}" (at 231.14 231.14 0) (fields_autoplaced)
     (effects (font (size 1.524 1.524)) (justify left bottom))
   )
@@
   (symbol (lib_name "BUSPC_HOST_5") (lib_id "isa_backplane-rescue:BUSPC_HOST") (at 127 157.48 180) (unit 1)
     (in_bom yes) (on_board yes) (dnp no)
-    (property "Reference" "BUS6" (at 111.76 115.57 0)
+    (property "Reference" "BUS8" (at 111.76 115.57 0)
       (effects (font (size 1.778 1.778)) (justify left))
     )
@@
       (project "isa_backplane"
         (path "/d4f5757f-f5cb-4873-a77e-cd912a261ecc"
-          (reference "BUS6") (unit 1)
+          (reference "BUS8") (unit 1)
         )
       )
@@
     )
   )
-  (symbol (lib_id "isa_backplane-rescue:RR5") (at 246.38 232.41 0) (unit 1)
-    (in_bom yes) (on_board yes) (dnp no)
-    (property "Reference" "RR5" (at 243.84 223.52 0)
-      (effects (font (size 1.27 1.27)) (justify left))
-    )
-    (property "Value" "4.7k" (at 243.84 241.3 0)
-      (effects (font (size 1.27 1.27)) (justify left))
-    )
-    (property "Footprint" "my_components:Conn_SIL6" (at 246.38 237.49 0)
-      (effects (font (size 1.27 1.27)) hide)
-    )
-    (property "Datasheet" "" (at 246.38 237.49 0)
-      (effects (font (size 1.27 1.27)))
-    )
-    (pin "1")
-    (pin "2")
-    (pin "3")
-    (pin "4")
-    (pin "5")
-    (pin "6")
-    (instances
-      (project "isa_backplane"
-        (path "/d4f5757f-f5cb-4873-a77e-cd912a261ecc"
-          (reference "RR5") (unit 1)
-        )
-      )
-    )
-  )
   (symbol (lib_id "isa_backplane-rescue:VCC") (at 276.86 134.62 0) (unit 1)
     (in_bom yes) (on_board yes) (dnp no)
@@
   (symbol (lib_id "isa_backplane-rescue:BUSPC_HOST") (at 200.66 157.48 180) (unit 1)
     (in_bom yes) (on_board yes) (dnp no)
-    (property "Reference" "BUS7" (at 185.42 115.57 0)
+    (property "Reference" "BUS9" (at 185.42 115.57 0)
       (effects (font (size 1.778 1.778)) (justify left))
     )
@@
       (project "isa_backplane"
         (path "/d4f5757f-f5cb-4873-a77e-cd912a261ecc"
-          (reference "BUS7") (unit 1)
+          (reference "BUS9") (unit 1)
         )
       )
@@
   (symbol (lib_name "BUSPC_DEV_1") (lib_id "isa_backplane-rescue:BUSPC_DEV") (at -111.76 63.5 180) (unit 1)
     (in_bom yes) (on_board yes) (dnp no)
-    (property "Reference" "BUS8" (at -127 21.59 0)
+    (property "Reference" "BUS6" (at -127 21.59 0)
       (effects (font (size 1.778 1.778)) (justify left))
     )
@@
       (project "isa_backplane"
         (path "/d4f5757f-f5cb-4873-a77e-cd912a261ecc"
-          (reference "BUS8") (unit 1)
+          (reference "BUS6") (unit 1)
+        )
+      )
+    )
+  )
+  (symbol (lib_id "my_components:RR4") (at 246.38 231.14 0) (unit 1)
+    (in_bom yes) (on_board yes) (dnp no) (fields_autoplaced)
+    (property "Reference" "RR5" (at 250.19 230.505 0)
+      (effects (font (size 1.27 1.27)) (justify left))
+    )
+    (property "Value" "4.7k" (at 250.19 233.045 0)
+      (effects (font (size 1.27 1.27)) (justify left))
+    )
+    (property "Footprint" "My_Components:Conn_SIL5" (at 246.38 237.49 0)
+      (effects (font (size 1.27 1.27)) hide)
+    )
+    (property "Datasheet" "" (at 246.38 237.49 0)
+      (effects (font (size 1.27 1.27)))
+    )
+    (pin "1")
+    (pin "2")
+    (pin "3")
+    (pin "4")
+    (pin "5")
+    (instances
+      (project "isa_backplane"
+        (path "/d4f5757f-f5cb-4873-a77e-cd912a261ecc"
+          (reference "RR5") (unit 1)
         )
       )
@@
   (symbol (lib_name "BUSPC_DEV_2") (lib_id "isa_backplane-rescue:BUSPC_DEV") (at -200.66 60.96 180) (unit 1)
     (in_bom yes) (on_board yes) (dnp no)
-    (property "Reference" "BUS9" (at -215.9 19.05 0)
+    (property "Reference" "BUS7" (at -215.9 19.05 0)
       (effects (font (size 1.778 1.778)) (justify left))
     )
@@
       (project "isa_backplane"
         (path "/d4f5757f-f5cb-4873-a77e-cd912a261ecc"
-          (reference "BUS9") (unit 1)
+          (reference "BUS7") (unit 1)
         )
       )
@@
         )
       )
+    )
+  )
+  (symbol (lib_id "isa_backplane-rescue:CP1") (at -107.95 246.38 0) (unit 1)
+    (in_bom yes) (on_board yes) (dnp no)
+    (property "Reference" "C28" (at -107.315 243.84 0)
+      (effects (font (size 1.27 1.27)) (justify left))
+    )
+    (property "Value" "10uF" (at -107.315 248.92 0)
+      (effects (font (size 1.27 1.27)) (justify left))
+    )
+    (property "Footprint" "My_Components:Cap_Tant_508" (at -107.95 246.38 0)
+      (effects (font (size 1.27 1.27)) hide)
+    )
+    (property "Datasheet" "" (at -107.95 246.38 0)
+      (effects (font (size 1.27 1.27)))
+    )
+    (pin "1")
+    (pin "2")
+    (instances
+      (project "isa_backplane"
+        (path "/d4f5757f-f5cb-4873-a77e-cd912a261ecc"
+          (reference "C28") (unit 1)
+        )
+      )

Commit message: Version 1.1
Parts:
- added HOLE10, HOLE9: HOLE, My_Components:Hole_4mm, symbol isa_backplane-rescue:HOLE
- BUS1, BUS2, BUS3, BUS4, BUS5, BUS8, BUS9: footprint my_components:Conn_Edge_ISA8 -> My_Components:Conn_Edge_ISA8
- C1, C10, C11, C12, C13, C14, C15, C16, C17, C18, C19, C2, C20, C3, C4, C5, C6, C7, C8, C9: footprint my_components:Cap_Tant_508 -> My_Components:Cap_Tant_508
- C21: footprint my_components:Cap_Cer_508 -> My_Components:Cap_Cer_762
- C22: footprint my_components:Cap_Cer_508 -> My_Components:Cap_Cer_508
- D1, D2: footprint my_components:LED_3mm -> My_Components:LED_3mm
- D3, D4: footprint my_components:Diode_762 -> My_Components:Diode_762
- HOLE1, HOLE2, HOLE3, HOLE4, HOLE5, HOLE6, HOLE7, HOLE8: footprint my_components:Hole_4mm -> My_Components:Hole_4mm
- P1: footprint my_components:Conn_Power_ATX_20pin -> My_Components:Conn_Power_ATX_20pin
- P2, P3: footprint my_components:Conn_Pin_Header_2x1_2.54mm -> My_Components:Conn_Pin_Header_2x1_2.54mm
- R1, R2, R3, R4, R5, R6, R7: footprint my_components:Res_762 -> My_Components:Res_762
- RR1, RR2, RR3: footprint my_components:Conn_SIL10 -> My_Components:Conn_SIL10
- RR4: footprint my_components:Conn_SIL6 -> My_Components:Conn_SIL6
- SW1: footprint my_components:Switch_Tactile_6mm -> My_Components:Switch_Tactile_6mm
- U1, U2: footprint my_components:IC_DIP14_300 -> My_Components:IC_DIP14_300
- U3: footprint my_components:IC_TO220-3_Horiz -> My_Components:IC_TO220-3_Vert
Connections:
- net GND: now also HOLE10.1, HOLE9.1
